File: Cad/FeelerBox1Eagle/feelerBox1.brd (EAGLE design)
At the start: 30 parts, among them IC1 4093N, Q1 BC640, Q2 2N2222A, Q5 BC640, Q6 2N2222A, T1 BC337

Commit message: fixes0.1
Parts:
- removed R13: (no value), SparkFun-Resistors:AXIAL-0.1
- added JP3: (no value), SparkFun:1X02
- added R7: (no value), SparkFun-Resistors:AXIAL-0.3
- moved R14 3.00 mm to (6.22, 46.4)
- moved VIB 3.00 mm to (5.97, 42.7)
- moved D1 3.00 mm to (9.45, 49.6)
- moved T1 2.06 mm to (17.5, 42.4), turned to 180 degrees
- moved C3 2.00 mm to (10.4, 41.7)
Connections:
- removed net N$22: C2.-, IC1.7, JP2.2, Q2.1
- new net BATTERYPWR: IC1.14, JP2.2, Q5.E, R11.P$2, R14.P$2, R2.P$2, R3.P$2
- net BATTERYGND: now also C2.-, IC1.7, JP1.2, JP3.1, Q2.1; no longer IC1.14, Q5.E, R11.P$2, R14.P$2, R2.P$2, R3.P$2
- net D2: now also R7.P$2; no longer R13.P$1
- net GND: no longer JP1.2
- net N$17: now also R7.P$1; no longer R13.P$2
- net N$6: now also JP3.2
Routing:
- net BATTERYPWR: track 0.00 -> 155.2 mm
- net N$22: track 149.5 -> 0.00 mm
- net N$20: track 10.2 -> 0.00 mm
- net N$6: track 9.50 -> 15.9 mm
- net D2: track 9.57 -> 14.5 mm
- net N$37: track 20.3 -> 23.1 mm
- net BATTERYGND: track 0.00 -> 1.39 mm
- net N$38: track 17.8 -> 18.7 mm
- net N$17: track 7.27 -> 6.70 mm
