File: Cad/FeelerBox1Eagle/box1LEDS.sch (EAGLE design)
At the start: 20 parts, among them Q3 2N2222A, Q4 2N2222A, Q5 2N2222A, X2 87758-0216

Commit message: fixes0.1
Parts:
- removed CN2: (no value), con-hdrs40:HDR-1X3-70543-?
- removed Q3, Q4, Q5: 2N2222A, transistor-npn:2N2222A
- removed R4, R5, R6: (no value), SparkFun-Passives:RESISTORPTH-1/4W
- removed X2: 87758-0216, con-molex:87758-0216
- added CN1: (no value), con-hdrs40:HDR-1X2-SIP-100
Connections:
- removed net D11: CN2.3, R6.1
- removed net D13: CN2.1, R4.2
- removed net N$29: Q3.C, U$6.-
- removed net N$31: Q4.C, U$5.-
- removed net N$32: Q5.C, U$4.-
- removed net N$6: Q3.E, Q4.E, Q5.E, X2-2.S
- removed net N$7: Q4.B, R5.2
- removed net N$8: CN2.2, R5.1
- removed net N$9: Q5.B, R4.1
- net N$4: now also CN1.2, U$4.-, U$5.-, U$6.-; no longer Q3.B, R6.2
- net N$5: now also CN1.1; no longer X2-1.S
Changed lines of the file:
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@@
 <part name="U$8" library="wh2001" deviceset="WS2001" device=""/>
 <part name="U$9" library="wh2001" deviceset="WS2001" device=""/>
-<part name="Q3" library="transistor-npn" deviceset="2N2222*" device="" technology="A"/>
-<part name="Q4" library="transistor-npn" deviceset="2N2222*" device="" technology="A"/>
-<part name="Q5" library="transistor-npn" deviceset="2N2222*" device="" technology="A"/>
 <part name="R1" library="SparkFun-Passives" deviceset="RESISTOR" device="PTH-1/4W"/>
 <part name="R2" library="SparkFun-Passives" deviceset="RESISTOR" device="PTH-1/4W"/>
 <part name="R3" library="SparkFun-Passives" deviceset="RESISTOR" device="PTH-1/4W"/>
-<part name="X2" library="con-molex" deviceset="87758-0216" device=""/>
-<part name="R4" library="SparkFun-Passives" deviceset="RESISTOR" device="PTH-1/4W"/>
-<part name="R5" library="SparkFun-Passives" deviceset="RESISTOR" device="PTH-1/4W"/>
-<part name="R6" library="SparkFun-Passives" deviceset="RESISTOR" device="PTH-1/4W"/>
-<part name="CN2" library="con-hdrs40" deviceset="HDR-1X3" device="-70543-?"/>
+<part name="CN1" library="con-hdrs40" deviceset="HDR-1X2" device="-SIP-100"/>
 </parts>
 <sheets>
@@
 <instance part="U$8" gate="G$1" x="15.24" y="68.58"/>
 <instance part="U$9" gate="G$1" x="33.02" y="68.58"/>
-<instance part="Q3" gate="G$1" x="30.48" y="15.24"/>
-<instance part="Q4" gate="G$1" x="12.7" y="15.24"/>
-<instance part="Q5" gate="G$1" x="-5.08" y="15.24"/>
 <instance part="R1" gate="G$1" x="-2.54" y="93.98" rot="R90"/>
 <instance part="R2" gate="G$1" x="15.24" y="93.98" rot="R90"/>
 <instance part="R3" gate="G$1" x="33.02" y="93.98" rot="R90"/>
-<instance part="X2" gate="-1" x="0" y="134.62"/>
-<instance part="X2" gate="-2" x="22.86" y="134.62" rot="R180"/>
-<instance part="R4" gate="G$1" x="-12.7" y="15.24" rot="R180"/>
-<instance part="R5" gate="G$1" x="10.16" y="10.16" rot="R90"/>
-<instance part="R6" gate="G$1" x="27.94" y="10.16" rot="R90"/>
-<instance part="CN2" gate="G$1" x="-33.02" y="109.22"/>
+<instance part="CN1" gate="G$1" x="-2.54" y="139.7" rot="R90"/>
 </instances>
 <busses>
 </busses>
 <nets>
-<net name="D13" class="0">
-<segment>
-<wire x1="-17.78" y1="15.24" x2="-66.04" y2="15.24" width="0.1524" layer="91"/>
-<wire x1="-66.04" y1="15.24" x2="-66.04" y2="111.76" width="0.1524" layer="91"/>
-<pinref part="R4" gate="G$1" pin="2"/>
-<pinref part="CN2" gate="G$1" pin="1"/>
-<wire x1="-38.1" y1="111.76" x2="-66.04" y2="111.76" width="0.1524" layer="91"/>
-</segment>
-</net>
 <net name="N$20" class="0">
 <segment>
@@
 </segment>
 </net>
-<net name="N$29" class="0">
-<segment>
-<pinref part="U$6" gate="G$1" pin="-"/>
-<pinref part="Q3" gate="G$1" pin="C"/>
-</segment>
-</net>
-<net name="N$31" class="0">
-<segment>
-<pinref part="U$5" gate="G$1" pin="-"/>
-<pinref part="Q4" gate="G$1" pin="C"/>
-</segment>
-</net>
-<net name="N$32" class="0">
-<segment>
-<pinref part="U$4" gate="G$1" pin="-"/>
-<pinref part="Q5" gate="G$1" pin="C"/>
-</segment>
-</net>
-<net name="D11" class="0">
-<segment>
-<wire x1="27.94" y1="5.08" x2="27.94" y2="-7.62" width="0.1524" layer="91"/>
-<wire x1="27.94" y1="-7.62" x2="-71.12" y2="-7.62" width="0.1524" layer="91"/>
-<wire x1="-71.12" y1="-7.62" x2="-71.12" y2="106.68" width="0.1524" layer="91"/>
-<pinref part="R6" gate="G$1" pin="1"/>
-<pinref part="CN2" gate="G$1" pin="3"/>
-<wire x1="-38.1" y1="106.68" x2="-71.12" y2="106.68" width="0.1524" layer="91"/>
-</segment>
-</net>
 <net name="N$1" class="0">
 <segment>
@@
 <wire x1="-2.54" y1="99.06" x2="15.24" y2="99.06" width="0.1524" layer="91"/>
 <wire x1="-2.54" y1="99.06" x2="-2.54" y2="134.62" width="0.1524" layer="91"/>
-<pinref part="X2" gate="-1" pin="S"/>
-</segment>
-</net>
-<net name="N$6" class="0">
-<segment>
-<pinref part="Q5" gate="G$1" pin="E"/>
-<wire x1="-2.54" y1="10.16" x2="-2.54" y2="0" width="0.1524" layer="91"/>
-<wire x1="-2.54" y1="0" x2="15.24" y2="0" width="0.1524" layer="91"/>
-<pinref part="Q4" gate="G$1" pin="E"/>
-<wire x1="15.24" y1="0" x2="15.24" y2="10.16" width="0.1524" layer="91"/>
-<wire x1="15.24" y1="0" x2="33.02" y2="0" width="0.1524" layer="91"/>
-<pinref part="Q3" gate="G$1" pin="E"/>
-<wire x1="33.02" y1="0" x2="33.02" y2="10.16" width="0.1524" layer="91"/>
-<wire x1="33.02" y1="0" x2="43.18" y2="0" width="0.1524" layer="91"/>
-<wire x1="43.18" y1="0" x2="43.18" y2="134.62" width="0.1524" layer="91"/>
-<pinref part="X2" gate="-2" pin="S"/>
-<wire x1="43.18" y1="134.62" x2="25.4" y2="134.62" width="0.1524" layer="91"/>
-</segment>
-</net>
-<net name="N$8" class="0">
-<segment>
-<wire x1="10.16" y1="5.08" x2="10.16" y2="-5.08" width="0.1524" layer="91"/>
-<wire x1="10.16" y1="-5.08" x2="-68.58" y2="-5.08" width="0.1524" layer="91"/>
-<wire x1="-68.58" y1="-5.08" x2="-68.58" y2="109.22" width="0.1524" layer="91"/>
-<pinref part="R5" gate="G$1" pin="1"/>
-<pinref part="CN2" gate="G$1" pin="2"/>
-<wire x1="-38.1" y1="109.22" x2="-68.58" y2="109.22" width="0.1524" layer="91"/>
+<pinref part="CN1" gate="G$1" pin="1"/>
 </segment>
 </net>
 <net name="N$4" class="0">
 <segment>
-<pinref part="Q3" gate="G$1" pin="B"/>
-<pinref part="R6" gate="G$1" pin="2"/>
+<pinref part="CN1" gate="G$1" pin="2"/>
+<wire x1="0" y1="134.62" x2="50.8" y2="134.62" width="0.1524" layer="91"/>
+<wire x1="50.8" y1="134.62" x2="50.8" y2="20.32" width="0.1524" layer="91"/>
+<pinref part="U$6" gate="G$1" pin="-"/>
+<wire x1="50.8" y1="20.32" x2="33.02" y2="20.32" width="0.1524" layer="91"/>
+<pinref part="U$5" gate="G$1" pin="-"/>
+<wire x1="33.02" y1="20.32" x2="15.24" y2="20.32" width="0.1524" layer="91"/>
+<pinref part="U$4" gate="G$1" pin="-"/>
+<wire x1="15.24" y1="20.32" x2="-2.54" y2="20.32" width="0.1524" layer="91"/>
 </segment>
 </net>
-<net name="N$7" class="0">
-<segment>
-<pinref part="Q4" gate="G$1" pin="B"/>
-<pinref part="R5" gate="G$1" pin="2"/>
-</segment>
-</net>
-<net name="N$9" class="0">
-<segment>
-<pinref part="Q5" gate="G$1" pin="B"/>
-<pinref part="R4" gate="G$1" pin="1"/>
-</segment>
-</net>

Commit message: updates
bah
Connections:
- removed net N$20: U$1.+, U$7.-
- removed net N$21: U$2.+, U$8.-
- removed net N$22: U$3.+, U$9.-
- removed net N$23: U$3.-, U$6.+
- removed net N$24: U$2.-, U$5.+
- removed net N$25: U$1.-, U$4.+
- removed net N$4: CN1.2, U$4.-, U$5.-, U$6.-
- new net GND: CN1.2, U$1.-, U$2.-, U$3.-, U$4.-, U$5.-, U$6.-, U$7.-, U$8.-, U$9.-
- net N$1: now also U$3.+, U$6.+
- net N$2: now also U$2.+, U$5.+
- net N$3: now also U$1.+, U$4.+
Other:
- moved on the sheet: CN1, R1, R3, U$1, U$2, U$3, U$4, U$5, U$6, U$7, U$9
Changed lines of the file:
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@@
 </plain>
 <instances>
-<instance part="U$1" gate="G$1" x="-2.54" y="48.26"/>
-<instance part="U$2" gate="G$1" x="15.24" y="48.26"/>
-<instance part="U$3" gate="G$1" x="33.02" y="48.26"/>
-<instance part="U$4" gate="G$1" x="-2.54" y="27.94"/>
-<instance part="U$5" gate="G$1" x="15.24" y="27.94"/>
-<instance part="U$6" gate="G$1" x="33.02" y="27.94"/>
-<instance part="U$7" gate="G$1" x="-2.54" y="68.58"/>
+<instance part="U$1" gate="G$1" x="-35.56" y="68.58"/>
+<instance part="U$2" gate="G$1" x="30.48" y="68.58"/>
+<instance part="U$3" gate="G$1" x="66.04" y="68.58"/>
+<instance part="U$4" gate="G$1" x="-48.26" y="68.58"/>
+<instance part="U$5" gate="G$1" x="2.54" y="68.58"/>
+<instance part="U$6" gate="G$1" x="50.8" y="68.58"/>
+<instance part="U$7" gate="G$1" x="-20.32" y="68.58"/>
 <instance part="U$8" gate="G$1" x="15.24" y="68.58"/>
-<instance part="U$9" gate="G$1" x="33.02" y="68.58"/>
-<instance part="R1" gate="G$1" x="-2.54" y="93.98" rot="R90"/>
+<instance part="U$9" gate="G$1" x="81.28" y="68.58"/>
+<instance part="R1" gate="G$1" x="-20.32" y="93.98" rot="R90"/>
 <instance part="R2" gate="G$1" x="15.24" y="93.98" rot="R90"/>
-<instance part="R3" gate="G$1" x="33.02" y="93.98" rot="R90"/>
-<instance part="CN1" gate="G$1" x="-2.54" y="139.7" rot="R90"/>
+<instance part="R3" gate="G$1" x="81.28" y="93.98" rot="R90"/>
+<instance part="CN1" gate="G$1" x="-20.32" y="139.7" rot="R90"/>
 </instances>
 <busses>
 </busses>
 <nets>
-<net name="N$20" class="0">
-<segment>
-<pinref part="U$1" gate="G$1" pin="+"/>
-<pinref part="U$7" gate="G$1" pin="-"/>
-<wire x1="-2.54" y1="55.88" x2="-2.54" y2="60.96" width="0.1524" layer="91"/>
-</segment>
-</net>
-<net name="N$21" class="0">
-<segment>
-<pinref part="U$2" gate="G$1" pin="+"/>
-<pinref part="U$8" gate="G$1" pin="-"/>
-<wire x1="15.24" y1="55.88" x2="15.24" y2="60.96" width="0.1524" layer="91"/>
-</segment>
-</net>
-<net name="N$22" class="0">
-<segment>
-<pinref part="U$3" gate="G$1" pin="+"/>
-<pinref part="U$9" gate="G$1" pin="-"/>
-<wire x1="33.02" y1="55.88" x2="33.02" y2="60.96" width="0.1524" layer="91"/>
-</segment>
-</net>
-<net name="N$23" class="0">
-<segment>
-<pinref part="U$6" gate="G$1" pin="+"/>
-<pinref part="U$3" gate="G$1" pin="-"/>
-<wire x1="33.02" y1="35.56" x2="33.02" y2="40.64" width="0.1524" layer="91"/>
-</segment>
-</net>
-<net name="N$24" class="0">
-<segment>
-<pinref part="U$5" gate="G$1" pin="+"/>
-<pinref part="U$2" gate="G$1" pin="-"/>
-<wire x1="15.24" y1="35.56" x2="15.24" y2="40.64" width="0.1524" layer="91"/>
-</segment>
-</net>
-<net name="N$25" class="0">
-<segment>
-<pinref part="U$4" gate="G$1" pin="+"/>
-<pinref part="U$1" gate="G$1" pin="-"/>
-<wire x1="-2.54" y1="35.56" x2="-2.54" y2="40.64" width="0.1524" layer="91"/>
-</segment>
-</net>
 <net name="N$1" class="0">
 <segment>
 <pinref part="U$9" gate="G$1" pin="+"/>
 <pinref part="R3" gate="G$1" pin="1"/>
-<wire x1="33.02" y1="76.2" x2="33.02" y2="88.9" width="0.1524" layer="91"/>
+<wire x1="81.28" y1="76.2" x2="81.28" y2="83.82" width="0.1524" layer="91"/>
+<pinref part="U$6" gate="G$1" pin="+"/>
+<wire x1="50.8" y1="76.2" x2="50.8" y2="83.82" width="0.1524" layer="91"/>
+<wire x1="50.8" y1="83.82" x2="66.04" y2="83.82" width="0.1524" layer="91"/>
+<wire x1="66.04" y1="83.82" x2="81.28" y2="83.82" width="0.1524" layer="91"/>
+<wire x1="81.28" y1="83.82" x2="81.28" y2="88.9" width="0.1524" layer="91"/>
+<pinref part="U$3" gate="G$1" pin="+"/>
+<wire x1="66.04" y1="76.2" x2="66.04" y2="83.82" width="0.1524" layer="91"/>
 </segment>
 </net>
@@
 <pinref part="U$8" gate="G$1" pin="+"/>
 <pinref part="R2" gate="G$1" pin="1"/>
-<wire x1="15.24" y1="76.2" x2="15.24" y2="88.9" width="0.1524" layer="91"/>
+<wire x1="15.24" y1="76.2" x2="15.24" y2="83.82" width="0.1524" layer="91"/>
+<pinref part="U$2" gate="G$1" pin="+"/>
+<wire x1="15.24" y1="83.82" x2="15.24" y2="88.9" width="0.1524" layer="91"/>
+<wire x1="15.24" y1="83.82" x2="30.48" y2="83.82" width="0.1524" layer="91"/>
+<wire x1="30.48" y1="83.82" x2="30.48" y2="76.2" width="0.1524" layer="91"/>
+<pinref part="U$5" gate="G$1" pin="+"/>
+<wire x1="15.24" y1="83.82" x2="2.54" y2="83.82" width="0.1524" layer="91"/>
+<wire x1="2.54" y1="83.82" x2="2.54" y2="76.2" width="0.1524" layer="91"/>
 </segment>
 </net>
@@
 <pinref part="U$7" gate="G$1" pin="+"/>
 <pinref part="R1" gate="G$1" pin="1"/>
-<wire x1="-2.54" y1="76.2" x2="-2.54" y2="88.9" width="0.1524" layer="91"/>
+<wire x1="-20.32" y1="76.2" x2="-20.32" y2="83.82" width="0.1524" layer="91"/>
+<wire x1="-20.32" y1="83.82" x2="-20.32" y2="88.9" width="0.1524" layer="91"/>
+<wire x1="-20.32" y1="83.82" x2="-35.56" y2="83.82" width="0.1524" layer="91"/>
+<pinref part="U$4" gate="G$1" pin="+"/>
+<wire x1="-35.56" y1="83.82" x2="-48.26" y2="83.82" width="0.1524" layer="91"/>
+<wire x1="-48.26" y1="83.82" x2="-48.26" y2="76.2" width="0.1524" layer="91"/>
+<pinref part="U$1" gate="G$1" pin="+"/>
+<wire x1="-35.56" y1="76.2" x2="-35.56" y2="83.82" width="0.1524" layer="91"/>
 </segment>
 </net>
@@
 <pinref part="R3" gate="G$1" pin="2"/>
 <pinref part="R2" gate="G$1" pin="2"/>
-<wire x1="33.02" y1="99.06" x2="15.24" y2="99.06" width="0.1524" layer="91"/>
+<wire x1="81.28" y1="99.06" x2="15.24" y2="99.06" width="0.1524" layer="91"/>
 <pinref part="R1" gate="G$1" pin="2"/>
-<wire x1="-2.54" y1="99.06" x2="15.24" y2="99.06" width="0.1524" layer="91"/>
-<wire x1="-2.54" y1="99.06" x2="-2.54" y2="134.62" width="0.1524" layer="91"/>
+<wire x1="-20.32" y1="99.06" x2="15.24" y2="99.06" width="0.1524" layer="91"/>
+<wire x1="-20.32" y1="99.06" x2="-20.32" y2="134.62" width="0.1524" layer="91"/>
 <pinref part="CN1" gate="G$1" pin="1"/>
 </segment>
 </net>
-<net name="N$4" class="0">
+<net name="GND" class="0">
 <segment>
 <pinref part="CN1" gate="G$1" pin="2"/>
-<wire x1="0" y1="134.62" x2="50.8" y2="134.62" width="0.1524" layer="91"/>
-<wire x1="50.8" y1="134.62" x2="50.8" y2="20.32" width="0.1524" layer="91"/>
+<wire x1="-17.78" y1="134.62" x2="88.9" y2="134.62" width="0.1524" layer="91"/>
+<wire x1="88.9" y1="134.62" x2="88.9" y2="20.32" width="0.1524" layer="91"/>
+<pinref part="U$4" gate="G$1" pin="-"/>
+<wire x1="-48.26" y1="60.96" x2="-45.72" y2="60.96" width="0.1524" layer="91"/>
+<wire x1="-45.72" y1="60.96" x2="-45.72" y2="20.32" width="0.1524" layer="91"/>
+<wire x1="-45.72" y1="20.32" x2="-35.56" y2="20.32" width="0.1524" layer="91"/>
+<pinref part="U$1" gate="G$1" pin="-"/>
+<wire x1="-35.56" y1="20.32" x2="-20.32" y2="20.32" width="0.1524" layer="91"/>
+<wire x1="-20.32" y1="20.32" x2="2.54" y2="20.32" width="0.1524" layer="91"/>
+<wire x1="2.54" y1="20.32" x2="15.24" y2="20.32" width="0.1524" layer="91"/>
+<wire x1="15.24" y1="20.32" x2="30.48" y2="20.32" width="0.1524" layer="91"/>
+<wire x1="30.48" y1="20.32" x2="50.8" y2="20.32" width="0.1524" layer="91"/>
+<wire x1="50.8" y1="20.32" x2="66.04" y2="20.32" width="0.1524" layer="91"/>
+<wire x1="66.04" y1="20.32" x2="81.28" y2="20.32" width="0.1524" layer="91"/>
+<wire x1="81.28" y1="20.32" x2="88.9" y2="20.32" width="0.1524" layer="91"/>
+<wire x1="-35.56" y1="60.96" x2="-35.56" y2="20.32" width="0.1524" layer="91"/>
+<pinref part="U$7" gate="G$1" pin="-"/>
+<wire x1="-20.32" y1="60.96" x2="-20.32" y2="20.32" width="0.1524" layer="91"/>
+<pinref part="U$5" gate="G$1" pin="-"/>
+<wire x1="2.54" y1="60.96" x2="2.54" y2="20.32" width="0.1524" layer="91"/>
+<pinref part="U$8" gate="G$1" pin="-"/>
+<wire x1="15.24" y1="60.96" x2="15.24" y2="20.32" width="0.1524" layer="91"/>
+<pinref part="U$2" gate="G$1" pin="-"/>
+<wire x1="30.48" y1="60.96" x2="30.48" y2="20.32" width="0.1524" layer="91"/>
+<pinref part="U$3" gate="G$1" pin="-"/>
+<wire x1="66.04" y1="60.96" x2="66.04" y2="20.32" width="0.1524" layer="91"/>
+<pinref part="U$9" gate="G$1" pin="-"/>
+<wire x1="81.28" y1="60.96" x2="81.28" y2="20.32" width="0.1524" layer="91"/>
 <pinref part="U$6" gate="G$1" pin="-"/>
-<wire x1="50.8" y1="20.32" x2="33.02" y2="20.32" width="0.1524" layer="91"/>
-<pinref part="U$5" gate="G$1" pin="-"/>
-<wire x1="33.02" y1="20.32" x2="15.24" y2="20.32" width="0.1524" layer="91"/>
-<pinref part="U$4" gate="G$1" pin="-"/>
-<wire x1="15.24" y1="20.32" x2="-2.54" y2="20.32" width="0.1524" layer="91"/>
+<wire x1="50.8" y1="60.96" x2="50.8" y2="20.32" width="0.1524" layer="91"/>
 </segment>
 </net>
